Commit message: updated allegro_kdl_xela.urdf

File: src/ll4ma_robots_description/urdf/allegro_right/allegro_kdl_xela.urdf (robot description, URDF)
Before this commit: robot allegro_hand_right, 22 links, 21 joints
Links:
- link index_link_1: mass 0.119 -> 0.159
- link index_link_2: mass 0.0847 -> 0.1147
- link index_tip: mass 0.0481 -> 0.0681
- link middle_link_1: mass 0.119 -> 0.159
- link middle_link_2: mass 0.0847 -> 0.1147
- link middle_tip: mass 0.0481 -> 0.0681
- link ring_link_1: mass 0.119 -> 0.159
- link ring_link_2: mass 0.0847 -> 0.1147
- link ring_tip: mass 0.0481 -> 0.0681
- link thumb_tip: mass 0.0268 -> 0.0468
